File: ST-Link V2.1.sch (KiCad schematic (older format))
At the start: 48 parts, among them J1 Conn_01x08, J2 USB_OTG, J4 Conn_01x08, Q1 MMBT3904, U0 stm32, U1 MIC5219-3.3, U2 USBLC6-2SC6, X1 8MHz

Commit message: duh
Connections:
- wire segments 161 -> 168
Changed lines of the file:
@@
 EESchema Schematic File Version 2
+LIBS:USBLC6-2SC6
 LIBS:power
 LIBS:device
@@
 NoConn ~ 4150 1800
 NoConn ~ 5800 2750
-$Comp
-L USBLC6-2SC6 U2
-U 1 1 59DF1810
-P 3650 6000
-F 0 "U2" H 3650 5700 60  0000 C CNN
-F 1 "USBLC6-2SC6" H 3650 6350 60  0000 C CNN
-F 2 "" H 3650 6000 60  0001 C CNN
-F 3 "" H 3650 6000 60  0001 C CNN
-	1    3650 6000
-	1    0    0    -1
-$EndComp
-Wire Wire Line
-	3200 5900 3200 5800
-Wire Wire Line
-	3200 5950 3100 5950
+Wire Wire Line
+	3100 5950 3250 5950
 Wire Wire Line
 	3100 5950 3100 6350
@@
 3V3_ST_LINK
 Wire Wire Line
-	4150 5950 4250 5950
+	3950 5950 4250 5950
 Wire Wire Line
 	4250 5950 4250 6550
 Text Label 4250 6550 0    60   ~ 0
 3V3_ST_LINK
+$Comp
+L USBLC6-2SC6 U2
+U 1 1 59DCEBAC
+P 3700 6050
+F 0 "U2" H 3600 5900 60  0000 C CNN
+F 1 "USBLC6-2SC6" H 3650 6400 60  0000 C CNN
+F 2 "" H 3700 6050 60  0001 C CNN
+F 3 "" H 3700 6050 60  0001 C CNN
+	1    3700 6050
+	1    0    0    -1
+$EndComp
+Wire Wire Line
+	3200 5900 3200 5850
+Wire Wire Line
+	3200 5850 3250 5850
+Wire Wire Line
+	3200 6100 3200 6050
+Wire Wire Line
+	3200 6050 3250 6050
+Wire Wire Line
+	3950 5850 4150 5850
+Wire Wire Line
+	4150 5850 4150 5800
+Wire Wire Line
+	3950 6050 4150 6050
+Wire Wire Line
+	4150 6050 4150 6100
 $EndSCHEMATC

Commit message: ROUTE RESISTOR
Parts:
- J1, J4: footprint Socket_Strips:Socket_Strip_Angled_1x08_Pitch2.54mm -> MetalPad:METAL_PAD
- U2: footprint (none) -> TO_SOT_Packages_SMD:SOT-23-6
Changed lines of the file:
@@
 F 0 "J1" H 9450 1500 50  0000 C CNN
 F 1 "Conn_01x08" H 9450 600 50  0000 C CNN
-F 2 "Socket_Strips:Socket_Strip_Angled_1x08_Pitch2.54mm" H 9450 1100 50  0001 C CNN
+F 2 "MetalPad:METAL_PAD" H 9450 1100 50  0001 C CNN
 F 3 "" H 9450 1100 50  0001 C CNN
 	1    9450 1100
@@
 F 0 "J4" H 9900 1500 50  0000 C CNN
 F 1 "Conn_01x08" H 9900 600 50  0000 C CNN
-F 2 "Socket_Strips:Socket_Strip_Angled_1x08_Pitch2.54mm" H 9900 1100 50  0001 C CNN
+F 2 "MetalPad:METAL_PAD" H 9900 1100 50  0001 C CNN
 F 3 "" H 9900 1100 50  0001 C CNN
 	1    9900 1100
@@
 F 0 "U2" H 3600 5900 60  0000 C CNN
 F 1 "USBLC6-2SC6" H 3650 6400 60  0000 C CNN
-F 2 "" H 3700 6050 60  0001 C CNN
+F 2 "TO_SOT_Packages_SMD:SOT-23-6" H 3700 6050 60  0001 C CNN
 F 3 "" H 3700 6050 60  0001 C CNN
 	1    3700 6050

Commit message: left abit
Parts:
- removed C12: 1uF, Capacitors_SMD:C_0603, symbol C
- removed R1: 0, Resistors_SMD:R_0603_HandSoldering, symbol R
- removed R15: 4.7K, Resistors_SMD:R_0603_HandSoldering, symbol R
- removed R26: 10K, Resistors_SMD:R_0603_HandSoldering, symbol R
- removed R27: [NA], Resistors_SMD:R_0603_HandSoldering, symbol R
- added J3: Conn_01x06, Socket_Strips:Socket_Strip_Straight_1x06_Pitch2.54mm, symbol Conn_01x06
- R22: value 100 -> 20
- U1: footprint TO_SOT_Packages_SMD:SOT-23-5 -> UFQFPN48:UFQFPN48
Connections:
- net labels added: GND, PC13, STM_SWCLK_JTCK, STM_SWDIO_JTMS, T_RESET, T_SWCLK_JTCK, T_SWDIO_JTMS, T_SWIM
- net labels removed: GNDREF, RESET, STM_JTCK, STM_JTMS, ST_LINK_SWIM, T_JTCK, T_JTMS
- wire segments 168 -> 155
- no-connect marks 16 -> 14
Other:
- moved on the sheet: C11, R11, R12, R13, R19, R20, R21

Commit message: working footprint(need to reroute)
Parts:
- C1: renamed from C18; footprint Capacitors_SMD:C_0603 -> Capacitors_SMD:C_0603_HandSoldering
- C10: renamed from C13; footprint Capacitors_SMD:C_0603 -> Capacitors_SMD:C_0603_HandSoldering
- C2: renamed from C7; footprint Capacitors_SMD:C_0603 -> Capacitors_SMD:C_0603_HandSoldering
- C3: renamed from C6; footprint Capacitors_SMD:C_0603 -> Capacitors_SMD:C_0603_HandSoldering
- C4: renamed from C15; footprint Capacitors_SMD:C_0603 -> Capacitors_SMD:C_0805_HandSoldering
- C5: renamed from C17; footprint Capacitors_SMD:C_0603 -> Capacitors_SMD:C_0805_HandSoldering
- C6: renamed from C8; footprint Capacitors_SMD:C_0603 -> Capacitors_SMD:C_0805_HandSoldering
- C7: renamed from C16; footprint Capacitors_SMD:C_0603 -> Capacitors_SMD:C_0603_HandSoldering
- C8: renamed from C5; footprint Capacitors_SMD:C_0603 -> Capacitors_SMD:C_0805_HandSoldering
- C9: renamed from C14; footprint Capacitors_SMD:C_0603 -> Capacitors_SMD:C_0603_HandSoldering
- renumbered J2 to J1, J3 to J2, J1 to J3, LD2 to LD1, R31 to R1, R14 to R10, R10 to R11, R3 to R12, R2 to R13, R11 to R14, R22 to R15, R4 to R16, R20 to R17, R21 to R18, R12 to R19, R29 to R2, R13 to R20, R19 to R21, R30 to R3, R7 to R4, R8 to R5, R5 to R7, R9 to R8, R23 to R9, U2 to U1, U0 to U2, U1 to U3
Other:
- moved on the sheet: R17, R18, R19, R20, R21

Commit message: routing
Parts:
- removed LD1: LED,RED, LEDs:LED_0603, symbol LED
- added D3: LED, LEDs:LED_0603, symbol LED
- C1, C10, C2, C3, C7, C9: footprint Capacitors_SMD:C_0603_HandSoldering -> Capacitors_SMD:C_0603
- C4, C5, C6, C8: footprint Capacitors_SMD:C_0805_HandSoldering -> Capacitors_SMD:C_0805
- R1, R10, R11, R14, R15, R16, R19, R2, R20, R21, R3, R4, R5, R6, R7, R8, R9: footprint Resistors_SMD:R_0603_HandSoldering -> Resistors_SMD:R_0603
- R12, R13, R17, R18: footprint Resistors_SMD:R_0603_HandSoldering -> Resistors_SMD:R_0805
- U3: footprint UFQFPN48:UFQFPN48 -> TO_SOT_Packages_SMD:SOT-23-5
Changed lines of the file:
@@
 LIBS:valves
 LIBS:ss
+LIBS:ST-Link V2.1-cache
 EELAYER 25 0
 EELAYER END
@@
 F 0 "C3" H 1525 2300 50  0000 L CNN
 F 1 "20pF" H 1525 2100 50  0000 L CNN
-F 2 "Capacitors_SMD:C_0603_HandSoldering" H 1538 2050 50  0001 C CNN
+F 2 "Capacitors_SMD:C_0603" H 1538 2050 50  0001 C CNN
 F 3 "" H 1500 2200 50  0001 C CNN
 	1    1500 2200
@@
 F 0 "C2" H 1125 2300 50  0000 L CNN
 F 1 "20pF" H 1125 2100 50  0000 L CNN
-F 2 "Capacitors_SMD:C_0603_HandSoldering" H 1138 2050 50  0001 C CNN
+F 2 "Capacitors_SMD:C_0603" H 1138 2050 50  0001 C CNN
 F 3 "" H 1100 2200 50  0001 C CNN
 	1    1100 2200
@@
 F 0 "R1" V 1080 2800 50  0000 C CNN
 F 1 "100K" V 1000 2800 50  0000 C CNN
-F 2 "Resistors_SMD:R_0603_HandSoldering" V 930 2800 50  0001 C CNN
+F 2 "Resistors_SMD:R_0603" V 930 2800 50  0001 C CNN
 F 3 "" H 1000 2800 50  0001 C CNN
 	1    1000 2800
@@
 F 0 "C1" H 1025 3500 50  0000 L CNN
 F 1 "100nF" H 1025 3300 50  0000 L CNN
-F 2 "Capacitors_SMD:C_0603_HandSoldering" H 1038 3250 50  0001 C CNN
+F 2 "Capacitors_SMD:C_0603" H 1038 3250 50  0001 C CNN
 F 3 "" H 1000 3400 50  0001 C CNN
 	1    1000 3400
@@
 F 0 "R14" V 5630 3700 50  0000 C CNN
 F 1 "100" V 5550 3700 50  0000 C CNN
-F 2 "Resistors_SMD:R_0603_HandSoldering" V 5480 3700 50  0001 C CNN
+F 2 "Resistors_SMD:R_0603" V 5480 3700 50  0001 C CNN
 F 3 "" H 5550 3700 50  0001 C CNN
 	1    5550 3700
@@
 F 0 "R10" V 3230 1200 50  0000 C CNN
 F 1 "100K" V 3150 1200 50  0000 C CNN
-F 2 "Resistors_SMD:R_0603_HandSoldering" V 3080 1200 50  0001 C CNN
+F 2 "Resistors_SMD:R_0603" V 3080 1200 50  0001 C CNN
 F 3 "" H 3150 1200 50  0001 C CNN
 	1    3150 1200
@@
 F 0 "C4" H 5175 5750 50  0000 L CNN
 F 1 "100nF" H 5175 5550 50  0000 L CNN
-F 2 "Capacitors_SMD:C_0805_HandSoldering" H 5188 5500 50  0001 C CNN
+F 2 "Capacitors_SMD:C_0805" H 5188 5500 50  0001 C CNN
 F 3 "" H 5150 5650 50  0001 C CNN
 	1    5150 5650
@@
 F 0 "C5" H 5475 5750 50  0000 L CNN
 F 1 "100nF" H 5475 5550 50  0000 L CNN
-F 2 "Capacitors_SMD:C_0805_HandSoldering" H 5488 5500 50  0001 C CNN
+F 2 "Capacitors_SMD:C_0805" H 5488 5500 50  0001 C CNN
 F 3 "" H 5450 5650 50  0001 C CNN
 	1    5450 5650
@@
 F 0 "C6" H 5725 5750 50  0000 L CNN
 F 1 "100nF" H 5725 5550 50  0000 L CNN
-F 2 "Capacitors_SMD:C_0805_HandSoldering" H 5738 5500 50  0001 C CNN
+F 2 "Capacitors_SMD:C_0805" H 5738 5500 50  0001 C CNN
 F 3 "" H 5700 5650 50  0001 C CNN
 	1    5700 5650
@@
 F 0 "C8" H 5975 5750 50  0000 L CNN
 F 1 "100nF" H 5975 5550 50  0000 L CNN
-F 2 "Capacitors_SMD:C_0805_HandSoldering" H 5988 5500 50  0001 C CNN
+F 2 "Capacitors_SMD:C_0805" H 5988 5500 50  0001 C CNN
 F 3 "" H 5950 5650 50  0001 C CNN
 	1    5950 5650
@@
 F 0 "R12" V 5130 6950 50  0000 C CNN
 F 1 "220" V 5050 6950 50  0000 C CNN
-F 2 "Resistors_SMD:R_0603_HandSoldering" V 4980 6950 50  0001 C CNN
+F 2 "Resistors_SMD:R_0805" V 4980 6950 50  0001 C CNN
 F 3 "" H 5050 6950 50  0001 C CNN
 	1    5050 6950
@@
 F 0 "R13" V 5130 7150 50  0000 C CNN
 F 1 "220" V 5050 7150 50  0000 C CNN
-F 2 "Resistors_SMD:R_0603_HandSoldering" V 4980 7150 50  0001 C CNN
+F 2 "Resistors_SMD:R_0805" V 4980 7150 50  0001 C CNN
 F 3 "" H 5050 7150 50  0001 C CNN
 	1    5050 7150
@@
 F 0 "R16" V 6880 5350 50  0000 C CNN
 F 1 "1K" V 6800 5350 50  0000 C CNN
-F 2 "Resistors_SMD:R_0603_HandSoldering" V 6730 5350 50  0001 C CNN
+F 2 "Resistors_SMD:R_0603" V 6730 5350 50  0001 C CNN
 F 3 "" H 6800 5350 50  0001 C CNN
 	1    6800 5350
 	-1   0    0    1
-$EndComp
-$Comp
-L LED LD1
-U 1 1 59D4648A
-P 6800 5750
-F 0 "LD1" H 6800 5850 50  0000 C CNN
-F 1 "LED,RED" H 6800 5650 50  0000 C CNN
-F 2 "LEDs:LED_0603" H 6800 5750 50  0001 C CNN
-F 3 "" H 6800 5750 50  0001 C CNN
-	1    6800 5750
-	0    -1   -1   0
 $EndComp
 $Comp
@@
 F 0 "R15" V 5680 3250 50  0000 C CNN
 F 1 "20" V 5600 3250 50  0000 C CNN
-F 2 "Resistors_SMD:R_0603_HandSoldering" V 5530 3250 50  0001 C CNN
+F 2 "Resistors_SMD:R_0603" V 5530 3250 50  0001 C CNN
 F 3 "" H 5600 3250 50  0001 C CNN
 	1    5600 3250
@@
 F 0 "C7" H 5875 3600 50  0000 L CNN
 F 1 "20pF" H 5875 3400 50  0000 L CNN
-F 2 "Capacitors_SMD:C_0603_HandSoldering" H 5888 3350 50  0001 C CNN
+F 2 "Capacitors_SMD:C_0603" H 5888 3350 50  0001 C CNN
 F 3 "" H 5850 3500 50  0001 C CNN
 	1    5850 3500
@@
 F 0 "R3" V 1680 3450 50  0000 C CNN
 F 1 "4K7" V 1600 3450 50  0000 C CNN
-F 2 "Resistors_SMD:R_0603_HandSoldering" V 1530 3450 50  0001 C CNN
+F 2 "Resistors_SMD:R_0603" V 1530 3450 50  0001 C CNN
 F 3 "" H 1600 3450 50  0001 C CNN
 	1    1600 3450
@@
 F 0 "R2" V 1580 3600 50  0000 C CNN
 F 1 "4K7" V 1500 3600 50  0000 C CNN
-F 2 "Resistors_SMD:R_0603_HandSoldering" V 1430 3600 50  0001 C CNN
+F 2 "Resistors_SMD:R_0603" V 1430 3600 50  0001 C CNN
 F 3 "" H 1500 3600 50  0001 C CNN
 	1    1500 3600
@@
 F 0 "R17" V 7690 3460 50  0000 C CNN
 F 1 "220" V 7610 3460 50  0000 C CNN
-F 2 "Resistors_SMD:R_0603_HandSoldering" V 7540 3460 50  0001 C CNN
+F 2 "Resistors_SMD:R_0805" V 7540 3460 50  0001 C CNN
 F 3 "" H 7610 3460 50  0001 C CNN
 	1    7610 3460
@@
 F 0 "R18" V 7690 3710 50  0000 C CNN
 F 1 "220" V 7610 3710 50  0000 C CNN
-F 2 "Resistors_SMD:R_0603_HandSoldering" V 7540 3710 50  0001 C CNN
+F 2 "Resistors_SMD:R_0805" V 7540 3710 50  0001 C CNN
 F 3 "" H 7610 3710 50  0001 C CNN
 	1    7610 3710
@@
 F 0 "R20" V 8440 3460 50  0000 C CNN
 F 1 "47" V 8360 3460 50  0000 C CNN
-F 2 "Resistors_SMD:R_0603_HandSoldering" V 8290 3460 50  0001 C CNN
+F 2 "Resistors_SMD:R_0603" V 8290 3460 50  0001 C CNN
 F 3 "" H 8360 3460 50  0001 C CNN
 	1    8360 3460
@@
 F 0 "R21" V 8440 3710 50  0000 C CNN
 F 1 "47" V 8360 3710 50  0000 C CNN
-F 2 "Resistors_SMD:R_0603_HandSoldering" V 8290 3710 50  0001 C CNN
+F 2 "Resistors_SMD:R_0603" V 8290 3710 50  0001 C CNN
 F 3 "" H 8360 3710 50  0001 C CNN
 	1    8360 3710
@@
 F 0 "U3" H 8550 5775 50  0000 C CNN
 F 1 "MIC5219-3.3" H 8700 5775 50  0000 L CNN
-F 2 "UFQFPN48:UFQFPN48" H 8700 5875 50  0001 C CNN
+F 2 "TO_SOT_Packages_SMD:SOT-23-5" H 8700 5875 50  0001 C CNN
 F 3 "" H 8700 5550 50  0001 C CNN
 	1    8700 5550
@@
 F 0 "C9" H 7775 5750 50  0000 L CNN
 F 1 "1uF" H 7775 5550 50  0000 L CNN
-F 2 "Capacitors_SMD:C_0603_HandSoldering" H 7788 5500 50  0001 C CNN
+F 2 "Capacitors_SMD:C_0603" H 7788 5500 50  0001 C CNN
 F 3 "" H 7750 5650 50  0001 C CNN
 	1    7750 5650
@@
 F 0 "C10" H 9175 5800 50  0000 L CNN
 F 1 "1uF" H 9175 5600 50  0000 L CNN
-F 2 "Capacitors_SMD:C_0603_HandSoldering" H 9188 5550 50  0001 C CNN
+F 2 "Capacitors_SMD:C_0603" H 9188 5550 50  0001 C CNN
 F 3 "" H 9150 5700 50  0001 C CNN
 	1    9150 5700
@@
 F 0 "R6" V 2180 5600 50  0000 C CNN
 F 1 "1K5" V 2100 5600 50  0000 C CNN
-F 2 "Resistors_SMD:R_0603_HandSoldering" V 2030 5600 50  0001 C CNN
+F 2 "Resistors_SMD:R_0603" V 2030 5600 50  0001 C CNN
 F 3 "" H 2100 5600 50  0001 C CNN
 	1    2100 5600
@@
 F 0 "R7" V 2280 6000 50  0000 C CNN
 F 1 "100K" V 2200 6000 50  0000 C CNN
-F 2 "Resistors_SMD:R_0603_HandSoldering" V 2130 6000 50  0001 C CNN
+F 2 "Resistors_SMD:R_0603" V 2130 6000 50  0001 C CNN
 F 3 "" H 2200 6000 50  0001 C CNN
 	1    2200 6000
@@
 F 0 "R4" V 2080 5800 50  0000 C CNN
 F 1 "20" V 2000 5800 50  0000 C CNN
-F 2 "Resistors_SMD:R_0603_HandSoldering" V 1930 5800 50  0001 C CNN
+F 2 "Resistors_SMD:R_0603" V 1930 5800 50  0001 C CNN
 F 3 "" H 2000 5800 50  0001 C CNN
 	1    2000 5800
@@
 F 0 "R5" V 2080 5900 50  0000 C CNN
 F 1 "20" V 2000 5900 50  0000 C CNN
-F 2 "Resistors_SMD:R_0603_HandSoldering" V 1930 5900 50  0001 C CNN
+F 2 "Resistors_SMD:R_0603" V 1930 5900 50  0001 C CNN
 F 3 "" H 2000 5900 50  0001 C CNN
 	1    2000 5900
@@
 F 0 "R11" V 3280 5350 50  0000 C CNN
 F 1 "100" V 3200 5350 50  0000 C CNN
-F 2 "Resistors_SMD:R_0603_HandSoldering" V 3130 5350 50  0001 C CNN
+F 2 "Resistors_SMD:R_0603" V 3130 5350 50  0001 C CNN
 F 3 "" H 3200 5350 50  0001 C CNN
 	1    3200 5350
@@
 F 0 "R9" V 2980 5700 50  0000 C CNN
 F 1 "36K" V 2900 5700 50  0000 C CNN
-F 2 "Resistors_SMD:R_0603_HandSoldering" V 2830 5700 50  0001 C CNN
+F 2 "Resistors_SMD:R_0603" V 2830 5700 50  0001 C CNN
 F 3 "" H 2900 5700 50  0001 C CNN
 	1    2900 5700
@@
 F 0 "R8" V 2980 5050 50  0000 C CNN
 F 1 "10K" V 2900 5050 50  0000 C CNN
-F 2 "Resistors_SMD:R_0603_HandSoldering" V 2830 5050 50  0001 C CNN
+F 2 "Resistors_SMD:R_0603" V 2830 5050 50  0001 C CNN
 F 3 "" H 2900 5050 50  0001 C CNN
 	1    2900 5050
@@
 F 0 "R19" V 8190 3160 50  0000 C CNN
 F 1 "680" V 8110 3160 50  0000 C CNN
-F 2 "Resistors_SMD:R_0603_HandSoldering" V 8040 3160 50  0001 C CNN
+F 2 "Resistors_SMD:R_0603" V 8040 3160 50  0001 C CNN
 F 3 "" H 8110 3160 50  0001 C CNN
 	1    8110 3160
@@
 Wire Wire Line
 	3200 5900 3200 6050
+$Comp
+L LED D3
+U 1 1 59E06D1D
+P 6800 5750
+F 0 "D3" H 6910 5710 50  0000 C CNN
+F 1 "LED" H 6800 5650 50  0000 C CNN
+F 2 "LEDs:LED_0603" H 6800 5750 50  0001 C CNN
+F 3 "" H 6800 5750 50  0001 C CNN
+	1    6800 5750
+	0    -1   -1   0
+$EndComp
 $EndSCHEMATC

Commit message: left 3v3 and gnd
Parts:
- added C12: 100nF, Capacitors_SMD:C_0603, symbol C
- C10, C9: value 1uF -> 22nF
- C11: value 1uF -> 10uF
- C4, C5, C6, C8: footprint Capacitors_SMD:C_0805 -> Capacitors_SMD:C_0603
- D1, D2, D3: footprint LEDs:LED_0603 -> LEDs:LED_0805
- R12, R13: value 220 -> 510; footprint Resistors_SMD:R_0805 -> Resistors_SMD:R_0603
- R16: value 1K -> 510
- R17, R18: footprint Resistors_SMD:R_0805 -> Resistors_SMD:R_0603
- R6: value 1K5 -> 4K7
Changed lines of the file:
@@
 F 0 "C4" H 5175 5750 50  0000 L CNN
 F 1 "100nF" H 5175 5550 50  0000 L CNN
-F 2 "Capacitors_SMD:C_0805" H 5188 5500 50  0001 C CNN
+F 2 "Capacitors_SMD:C_0603" H 5188 5500 50  0001 C CNN
 F 3 "" H 5150 5650 50  0001 C CNN
 	1    5150 5650
@@
 F 0 "C5" H 5475 5750 50  0000 L CNN
 F 1 "100nF" H 5475 5550 50  0000 L CNN
-F 2 "Capacitors_SMD:C_0805" H 5488 5500 50  0001 C CNN
+F 2 "Capacitors_SMD:C_0603" H 5488 5500 50  0001 C CNN
 F 3 "" H 5450 5650 50  0001 C CNN
 	1    5450 5650
@@
 F 0 "C6" H 5725 5750 50  0000 L CNN
 F 1 "100nF" H 5725 5550 50  0000 L CNN
-F 2 "Capacitors_SMD:C_0805" H 5738 5500 50  0001 C CNN
+F 2 "Capacitors_SMD:C_0603" H 5738 5500 50  0001 C CNN
 F 3 "" H 5700 5650 50  0001 C CNN
 	1    5700 5650
@@
 F 0 "C8" H 5975 5750 50  0000 L CNN
 F 1 "100nF" H 5975 5550 50  0000 L CNN
-F 2 "Capacitors_SMD:C_0805" H 5988 5500 50  0001 C CNN
+F 2 "Capacitors_SMD:C_0603" H 5988 5500 50  0001 C CNN
 F 3 "" H 5950 5650 50  0001 C CNN
 	1    5950 5650
@@
 P 5050 6950
 F 0 "R12" V 5130 6950 50  0000 C CNN
-F 1 "220" V 5050 6950 50  0000 C CNN
-F 2 "Resistors_SMD:R_0805" V 4980 6950 50  0001 C CNN
+F 1 "510" V 5050 6950 50  0000 C CNN
+F 2 "Resistors_SMD:R_0603" V 4980 6950 50  0001 C CNN
 F 3 "" H 5050 6950 50  0001 C CNN
 	1    5050 6950
@@
 P 5050 7150
 F 0 "R13" V 5130 7150 50  0000 C CNN
-F 1 "220" V 5050 7150 50  0000 C CNN
-F 2 "Resistors_SMD:R_0805" V 4980 7150 50  0001 C CNN
+F 1 "510" V 5050 7150 50  0000 C CNN
+F 2 "Resistors_SMD:R_0603" V 4980 7150 50  0001 C CNN
 F 3 "" H 5050 7150 50  0001 C CNN
 	1    5050 7150
@@
 P 6800 5350
 F 0 "R16" V 6880 5350 50  0000 C CNN
-F 1 "1K" V 6800 5350 50  0000 C CNN
+F 1 "510" V 6800 5350 50  0000 C CNN
 F 2 "Resistors_SMD:R_0603" V 6730 5350 50  0001 C CNN
 F 3 "" H 6800 5350 50  0001 C CNN
@@
 F 0 "R17" V 7690 3460 50  0000 C CNN
 F 1 "220" V 7610 3460 50  0000 C CNN
-F 2 "Resistors_SMD:R_0805" V 7540 3460 50  0001 C CNN
+F 2 "Resistors_SMD:R_0603" V 7540 3460 50  0001 C CNN
 F 3 "" H 7610 3460 50  0001 C CNN
 	1    7610 3460
@@
 F 0 "R18" V 7690 3710 50  0000 C CNN
 F 1 "220" V 7610 3710 50  0000 C CNN
-F 2 "Resistors_SMD:R_0805" V 7540 3710 50  0001 C CNN
+F 2 "Resistors_SMD:R_0603" V 7540 3710 50  0001 C CNN
 F 3 "" H 7610 3710 50  0001 C CNN
 	1    7610 3710
@@
 P 7750 5650
 F 0 "C9" H 7775 5750 50  0000 L CNN
-F 1 "1uF" H 7775 5550 50  0000 L CNN
+F 1 "22nF" H 7775 5550 50  0000 L CNN
 F 2 "Capacitors_SMD:C_0603" H 7788 5500 50  0001 C CNN
 F 3 "" H 7750 5650 50  0001 C CNN
@@
 P 9150 5700
 F 0 "C10" H 9175 5800 50  0000 L CNN
-F 1 "1uF" H 9175 5600 50  0000 L CNN
+F 1 "22nF" H 9175 5600 50  0000 L CNN
 F 2 "Capacitors_SMD:C_0603" H 9188 5550 50  0001 C CNN
 F 3 "" H 9150 5700 50  0001 C CNN
@@
 P 9530 5680
 F 0 "C11" H 9555 5780 50  0000 L CNN
-F 1 "1uF" H 9555 5580 50  0000 L CNN
+F 1 "10uF" H 9555 5580 50  0000 L CNN
 F 2 "Capacitors_SMD:C_0603" H 9568 5530 50  0001 C CNN
 F 3 "" H 9530 5680 50  0001 C CNN
@@
 P 2100 5600
 F 0 "R6" V 2180 5600 50  0000 C CNN
-F 1 "1K5" V 2100 5600 50  0000 C CNN
+F 1 "4K7" V 2100 5600 50  0000 C CNN
 F 2 "Resistors_SMD:R_0603" V 2030 5600 50  0001 C CNN
 F 3 "" H 2100 5600 50  0001 C CNN
@@
 Text Label 1450 3300 0    60   ~ 0
 3V3_ST_LINK
-Text Label 9520 5280 0    60   ~ 0
+Text Label 9530 5280 0    60   ~ 0
 3V3_ST_LINK
 Text Label 10500 1200 0    60   ~ 0
@@
 F 0 "D1" H 5800 7000 50  0000 C CNN
 F 1 "LED" H 5700 6850 50  0000 C CNN
-F 2 "LEDs:LED_0603" H 5700 6950 50  0001 C CNN
+F 2 "LEDs:LED_0805" H 5700 6950 50  0001 C CNN
 F 3 "" H 5700 6950 50  0001 C CNN
 	1    5700 6950
@@
 F 0 "D2" H 5810 7110 50  0000 C CNN
 F 1 "LED" H 5700 7050 50  0000 C CNN
-F 2 "LEDs:LED_0603" H 5700 7150 50  0001 C CNN
+F 2 "LEDs:LED_0805" H 5700 7150 50  0001 C CNN
 F 3 "" H 5700 7150 50  0001 C CNN
 	1    5700 7150
@@
 $EndComp
 Wire Wire Line
-	9000 5450 9530 5450
-Wire Wire Line
-	9530 5450 9530 5530
-Wire Wire Line
-	9520 5280 9520 5450
-Connection ~ 9520 5450
+	9000 5450 9990 5450
 $Comp
 L USBLC6-2SC6 U1
@@
 F 0 "D3" H 6910 5710 50  0000 C CNN
 F 1 "LED" H 6800 5650 50  0000 C CNN
-F 2 "LEDs:LED_0603" H 6800 5750 50  0001 C CNN
+F 2 "LEDs:LED_0805" H 6800 5750 50  0001 C CNN
 F 3 "" H 6800 5750 50  0001 C CNN
 	1    6800 5750
 	0    -1   -1   0
 $EndComp
+Wire Wire Line
+	9530 5280 9530 5530
+Connection ~ 9530 5450
+Wire Wire Line
+	9990 5450 9990 5520
+$Comp
+L C C12
+U 1 1 59E1553D
+P 9990 5670
+F 0 "C12" H 10015 5770 50  0000 L CNN
+F 1 "100nF" H 10015 5570 50  0000 L CNN
+F 2 "Capacitors_SMD:C_0603" H 10028 5520 50  0001 C CNN
+F 3 "" H 9990 5670 50  0001 C CNN
+	1    9990 5670
+	1    0    0    -1
+$EndComp
+$Comp
+L GND #PWR019
+U 1 1 59E156BB
+P 9990 5820
+F 0 "#PWR019" H 9990 5570 50  0001 C CNN
+F 1 "GND" H 9990 5670 50  0000 C CNN
+F 2 "" H 9990 5820 50  0001 C CNN
+F 3 "" H 9990 5820 50  0001 C CNN
+	1    9990 5820
+	1    0    0    -1
+$EndComp
 $EndSCHEMATC

Commit message: route route route
Parts:
- removed C7: 20pF, Capacitors_SMD:C_0603, symbol C
- removed R15: 20, Resistors_SMD:R_0603, symbol R
Connections:
- net labels added: STM_SWO, T_JRST, T_JTDI, T_JTDO
- net labels removed: MCO, PC13
- wire segments 155 -> 159
- no-connect marks 14 -> 9

Commit message: minor changes
Other:
- moved on the sheet: J2
Changed lines of the file:
@@
 L Conn_01x06 J2
 U 1 1 59DEFF36
-P 7320 1140
-F 0 "J2" H 7320 1440 50  0000 C CNN
-F 1 "Conn_01x06" H 7320 740 50  0000 C CNN
-F 2 "Socket_Strips:Socket_Strip_Straight_1x06_Pitch2.54mm" H 7320 1140 50  0001 C CNN
-F 3 "" H 7320 1140 50  0001 C CNN
-	1    7320 1140
-	1    0    0    -1
-$EndComp
-Text Label 6820 1040 2    60   ~ 0
+P 7720 1000
+F 0 "J2" H 7720 1300 50  0000 C CNN
+F 1 "Conn_01x06" H 7720 600 50  0000 C CNN
+F 2 "Socket_Strips:Socket_Strip_Straight_1x06_Pitch2.54mm" H 7720 1000 50  0001 C CNN
+F 3 "" H 7720 1000 50  0001 C CNN
+	1    7720 1000
+	1    0    0    -1
+$EndComp
+Text Label 7220 1200 2    60   ~ 0
 STM_SWCLK_JTCK
-Text Label 6820 1140 2    60   ~ 0
+Text Label 7220 1000 2    60   ~ 0
 STM_SWDIO_JTMS
-Text Label 6820 1240 2    60   ~ 0
+Text Label 7220 900  2    60   ~ 0
 NRST
-Text Label 6820 1340 2    60   ~ 0
+Text Label 7220 1100 2    60   ~ 0
 3V3_ST_LINK
 $Comp
@@
 L GND #PWR07
 U 1 1 59E1FDD5
-P 7120 940
-F 0 "#PWR07" H 7120 690 50  0001 C CNN
-F 1 "GND" H 7120 790 50  0000 C CNN
-F 2 "" H 7120 940 50  0001 C CNN
-F 3 "" H 7120 940 50  0001 C CNN
-	1    7120 940
+P 7520 800
+F 0 "#PWR07" H 7520 550 50  0001 C CNN
+F 1 "GND" H 7520 650 50  0000 C CNN
+F 2 "" H 7520 800 50  0001 C CNN
+F 3 "" H 7520 800 50  0001 C CNN
+	1    7520 800
 	0    1    1    0
 $EndComp
@@
 Text Label 9010 1300 2    60   ~ 0
 T_JRST
-Text Label 6820 1440 2    60   ~ 0
+Text Label 7220 1300 2    60   ~ 0
 STM_SWO
 Wire Wire Line
@@
 	5550 3900 5550 3850
 Wire Wire Line
-	7120 1040 6820 1040
-Wire Wire Line
-	7120 1140 6820 1140
-Wire Wire Line
-	7120 1240 6820 1240
-Wire Wire Line
-	7120 1340 6820 1340
-Wire Wire Line
-	7120 1440 6820 1440
+	7520 900  7220 900
+Wire Wire Line
+	7520 1000 7220 1000
+Wire Wire Line
+	7520 1100 7220 1100
+Wire Wire Line
+	7520 1200 7220 1200
+Wire Wire Line
+	7520 1300 7220 1300
 Wire Wire Line
 	7460 3710 6870 3710
