File: ST-Link V2.1.sch (KiCad schematic (older format))
At the start: 43 parts, among them J1 USB_OTG, J2 Conn_01x06, J3 Conn_01x08, J4 Conn_01x08, Q1 MMBT3904, U1 USBLC6-2SC6, U2 stm32, U3 MIC5219-3.3, X1 8MHz

Commit message: added 1C1R
Parts:
- added C7: 1uF, Capacitors_SMD:C_0603, symbol C
- added R15: 10K, Resistors_SMD:R_0603, symbol R
Connections:
- wire segments 159 -> 161
Changed lines of the file:
@@
 	4050 4050 4050 4600
 Connection ~ 4050 4300
+Text Label 1700 1200 0    60   ~ 0
+T_NRST
+$Comp
+L R R15
+U 1 1 59FDCA80
+P 1450 950
+F 0 "R15" V 1530 950 50  0000 C CNN
+F 1 "10K" V 1450 950 50  0000 C CNN
+F 2 "Resistors_SMD:R_0603" V 1380 950 50  0001 C CNN
+F 3 "" H 1450 950 50  0001 C CNN
+	1    1450 950
+	1    0    0    -1
+$EndComp
+$Comp
+L C C7
+U 1 1 59FDCAF3
+P 1450 1450
+F 0 "C7" H 1475 1550 50  0000 L CNN
+F 1 "1uF" H 1475 1350 50  0000 L CNN
+F 2 "Capacitors_SMD:C_0603" H 1488 1300 50  0001 C CNN
+F 3 "" H 1450 1450 50  0001 C CNN
+	1    1450 1450
+	1    0    0    -1
+$EndComp
+Wire Wire Line
+	1700 1200 1450 1200
+Connection ~ 1450 1200
+Wire Wire Line
+	1450 1100 1450 1300
+Text Label 1450 800  0    60   ~ 0
+3V3_ST_LINK
+$Comp
+L GND #PWR019
+U 1 1 59FDDE70
+P 1450 1600
+F 0 "#PWR019" H 1450 1350 50  0001 C CNN
+F 1 "GND" H 1450 1450 50  0000 C CNN
+F 2 "" H 1450 1600 50  0001 C CNN
+F 3 "" H 1450 1600 50  0001 C CNN
+	1    1450 1600
+	1    0    0    -1
+$EndComp
 $EndSCHEMATC

Commit message: checked schematic
Parts:
- removed C7: 1uF, Capacitors_SMD:C_0603, symbol C
- removed R15: 10K, Resistors_SMD:R_0603, symbol R
- added R22: 100K, Resistors_SMD:R_0603, symbol R
- added R23, R24: 10K, Resistors_SMD:R_0603, symbol R
- D1: value LED -> RED_LED
- D2: value LED -> BLUE_LED
Connections:
- wire segments 161 -> 163
- no-connect marks 9 -> 7
Changed lines of the file:
@@
 NoConn ~ 2550 2850
 NoConn ~ 3950 4050
-NoConn ~ 3750 4050
 NoConn ~ 3150 4050
 $Comp
@@
 P 5700 6950
 F 0 "D1" H 5800 7000 50  0000 C CNN
-F 1 "LED" H 5700 6850 50  0000 C CNN
+F 1 "RED_LED" H 5700 6850 50  0000 C CNN
 F 2 "LEDs:LED_0805" H 5700 6950 50  0001 C CNN
 F 3 "" H 5700 6950 50  0001 C CNN
@@
 P 5700 7150
 F 0 "D2" H 5810 7110 50  0000 C CNN
-F 1 "LED" H 5700 7050 50  0000 C CNN
+F 1 "BLUE_LED" H 5700 7050 50  0000 C CNN
 F 2 "LEDs:LED_0805" H 5700 7150 50  0001 C CNN
 F 3 "" H 5700 7150 50  0001 C CNN
@@
 	1    0    0    -1
 $EndComp
-NoConn ~ 2550 2650
 Text Label 3950 1660 1    60   ~ 0
 STM_SWO
@@
 	4150 4300 4350 4300
 Wire Wire Line
-	4150 4050 4150 4300
+	4150 4050 4150 4370
 Wire Wire Line
 	6800 5150 6800 5200
@@
 	1500 2350 1500 2950
 Wire Wire Line
-	3850 4300 4050 4300
-Wire Wire Line
 	3050 4650 3050 4050
 Wire Wire Line
@@
 	9250 1500 9010 1500
 Wire Wire Line
-	3850 4050 3850 4300
-Wire Wire Line
 	4050 4050 4050 4600
-Connection ~ 4050 4300
-Text Label 1700 1200 0    60   ~ 0
-T_NRST
-$Comp
-L R R15
-U 1 1 59FDCA80
-P 1450 950
-F 0 "R15" V 1530 950 50  0000 C CNN
-F 1 "10K" V 1450 950 50  0000 C CNN
-F 2 "Resistors_SMD:R_0603" V 1380 950 50  0001 C CNN
-F 3 "" H 1450 950 50  0001 C CNN
-	1    1450 950
-	1    0    0    -1
-$EndComp
-$Comp
-L C C7
-U 1 1 59FDCAF3
-P 1450 1450
-F 0 "C7" H 1475 1550 50  0000 L CNN
-F 1 "1uF" H 1475 1350 50  0000 L CNN
-F 2 "Capacitors_SMD:C_0603" H 1488 1300 50  0001 C CNN
-F 3 "" H 1450 1450 50  0001 C CNN
-	1    1450 1450
-	1    0    0    -1
-$EndComp
-Wire Wire Line
-	1700 1200 1450 1200
-Connection ~ 1450 1200
-Wire Wire Line
-	1450 1100 1450 1300
-Text Label 1450 800  0    60   ~ 0
-3V3_ST_LINK
+Wire Wire Line
+	3750 4050 3750 4300
+$Comp
+L R R22
+U 1 1 5A027035
+P 3750 4450
+F 0 "R22" V 3830 4450 50  0000 C CNN
+F 1 "100K" V 3750 4450 50  0000 C CNN
+F 2 "Resistors_SMD:R_0603" V 3680 4450 50  0001 C CNN
+F 3 "" H 3750 4450 50  0001 C CNN
+	1    3750 4450
+	-1   0    0    1
+$EndComp
+$Comp
+L R R23
+U 1 1 5A027C19
+P 3850 4220
+F 0 "R23" V 3930 4220 50  0000 C CNN
+F 1 "10K" V 3850 4220 50  0000 C CNN
+F 2 "Resistors_SMD:R_0603" V 3780 4220 50  0001 C CNN
+F 3 "" H 3850 4220 50  0001 C CNN
+	1    3850 4220
+	-1   0    0    1
+$EndComp
+Wire Wire Line
+	3850 4050 3850 4070
+Wire Wire Line
+	4150 4370 3850 4370
+Connection ~ 4150 4300
+Wire Wire Line
+	4050 4600 3750 4600
+$Comp
+L R R24
+U 1 1 5A02B4CB
+P 2100 2460
+F 0 "R24" V 2180 2460 50  0000 C CNN
+F 1 "10K" V 2100 2460 50  0000 C CNN
+F 2 "Resistors_SMD:R_0603" V 2030 2460 50  0001 C CNN
+F 3 "" H 2100 2460 50  0001 C CNN
+	1    2100 2460
+	-1   0    0    1
+$EndComp
+Wire Wire Line
+	2550 2650 2100 2650
+Wire Wire Line
+	2100 2650 2100 2610
 $Comp
 L GND #PWR019
-U 1 1 59FDDE70
-P 1450 1600
-F 0 "#PWR019" H 1450 1350 50  0001 C CNN
-F 1 "GND" H 1450 1450 50  0000 C CNN
-F 2 "" H 1450 1600 50  0001 C CNN
-F 3 "" H 1450 1600 50  0001 C CNN
-	1    1450 1600
-	1    0    0    -1
+U 1 1 5A02C087
+P 2100 2310
+F 0 "#PWR019" H 2100 2060 50  0001 C CNN
+F 1 "GND" H 2100 2160 50  0000 C CNN
+F 2 "" H 2100 2310 50  0001 C CNN
+F 3 "" H 2100 2310 50  0001 C CNN
+	1    2100 2310
+	-1   0    0    1
 $EndComp
 $EndSCHEMATC

Commit message: changed font and copper pour area
Changed lines of the file:
@@
 	1    0    0    -1
 $EndComp
-Text Label 3550 4450 1    60   ~ 0
+Text Label 3550 4650 1    60   ~ 0
 T_NRST
 Text Label 10500 900  0    60   ~ 0
@@
 	10100 900  10500 900
 Wire Wire Line
-	3550 4050 3550 4500
+	3550 4050 3550 4650
 Wire Wire Line
 	10100 800  10280 800
