File: ST-Link V2.1.kicad_pcb (KiCad board)
At the start: 2 copper layers, 33.6 x 21.1 mm, 45 parts, among them J1 USB_OTG, J2 Conn_01x06, J3 Conn_01x08, J4 Conn_01x08, Q1 MMBT3904, U1 USBLC6-2SC6, U2 stm32, U3 MIC5219-3.3, X1 8MHz

Commit message: save for reroute
Routing:
- net /T_SWIM: track 20.3 -> 16.4 mm
- net GND: track 124.5 -> 122.7 mm
- net /T_SWO: track 19.6 -> 18.3 mm
- net /T_SWDIO_JTMS: track 17.2 -> 16.1 mm
- net /T_SWCLK_JTCK: track 12.1 -> 11.3 mm
Other:
- net class Default: via_dia 0.4 -> 0.45

Commit message: route route route
Parts:
- removed C7: 20pF, Capacitors_SMD:C_0603
- removed R15: 20, Resistors_SMD:R_0603
- moved D3 3.09 mm to (126.3, 116.5)
- moved R16 1.52 mm to (127.5, 115.9)
- moved D2 1.43 mm to (144.4, 116.1)
- moved R13 1.43 mm to (144.4, 116.1)
- moved R14 1.19 mm to (140.6, 109.4)
- moved U1 1.16 mm to (124.4, 115.4)
- moved J3 1.15 mm to (148.3, 99.6)
- moved J4 1.15 mm to (148.3, 99.6)
- moved J2 1.13 mm to (143.5, 100.1)
- moved C12 1.13 mm to (137.9, 115.7)
- moved C8 1.13 mm to (136.3, 115.7)
- moved R1 1.13 mm to (131.5, 115.6)
- moved C1 1.13 mm to (129.8, 115.6)
- moved R3 1.13 mm to (133.1, 115.6)
- moved R2 1.13 mm to (134.7, 115.6)
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Connections:
- J2 pad 6: /PC13 -> /STM_SWO
- J3 pad 2: /T_SWIM -> /T_RESET
- J3 pad 3: Net-(J3-Pad3) -> /T_SWIM
- J3 pad 4: /T_RESET -> /3V3_ST_LINK
- J3 pad 5: /3V3_ST_LINK -> /PWR_ENn
- J3 pad 6: /PWR_ENn -> /T_JRST
- J3 pad 7: /MCO -> /T_JTDI
- J3 pad 8: Net-(J3-Pad8) -> /T_JTDO
- J4 pad 2: /T_SWCLK_JTCK -> /T_NRST
- J4 pad 4: /T_NRST -> /3V3_ST_LINK
- J4 pad 5: /3V3_ST_LINK -> /T_SWCLK_JTCK
- U2 pad 15: Net-(U2-Pad15) -> /T_SWCLK_JTCK
- U2 pad 16: Net-(U2-Pad16) -> /T_JTDO
- U2 pad 17: Net-(U2-Pad17) -> /T_JTDI
- U2 pad 19: Net-(U2-Pad19) -> /T_JRST
- U2 pad 2: /PC13 -> Net-(U2-Pad2)
- U2 pad 39: Net-(U2-Pad39) -> /STM_SWO
Routing:
- net GND: track 122.7 -> 0.00 mm, vias 16 -> 0
- net /3V3_ST_LINK: track 84.4 -> 0.00 mm, vias 20 -> 0
- net /NRST: track 36.4 -> 0.00 mm, vias 4 -> 0
- net +5V: track 22.3 -> 0.00 mm, vias 1 -> 0
- net /MCO: track 21.7 -> 0.00 mm, vias 3 -> 0
- net Net-(Q1-Pad2): track 15.9 -> 0.00 mm
- net /PC13: track 14.4 -> 0.00 mm, vias 1 -> 0
- net Net-(J1-Pad3): track 13.2 -> 0.00 mm, vias 3 -> 0
- net /USB_RENUMN: track 12.3 -> 0.00 mm, vias 1 -> 0
- net /T_NRST: track 11.8 -> 0.00 mm, vias 1 -> 0
- net /T_JTDO: track 0.00 -> 11.4 mm
- net /SWIM_RST_IN: track 10.1 -> 0.00 mm, vias 1 -> 0
- net Net-(C3-Pad2): track 9.69 -> 0.00 mm, vias 1 -> 0
- net /T_SWCLK_JTCK: track 11.3 -> 20.8 mm, vias 1 -> 2
- net Net-(J1-Pad2): track 9.49 -> 0.00 mm, vias 2 -> 0
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- removed copper zone on F.Cu, net /3V3_ST_LINK
- removed copper zone on B.Cu, net GND
Other:
- board size 33.6 x 21.1 mm -> 33.6 x 21.2 mm

Commit message: left 3.3 & gnd
Parts:
- turned C4 to 270 degrees
Routing:
- net GND: track 0.00 -> 47.1 mm, vias 0 -> 3
- net /NRST: track 0.00 -> 30.7 mm, vias 0 -> 2
- net /3V3_ST_LINK: track 0.00 -> 20.2 mm, vias 0 -> 3
- net /T_NRST: track 0.00 -> 17.7 mm, vias 0 -> 5
- net Net-(Q1-Pad2): track 0.00 -> 15.8 mm
- net /USB_RENUMN: track 0.00 -> 14.3 mm, vias 0 -> 1
- net Net-(J1-Pad3): track 0.00 -> 11.1 mm, vias 0 -> 1
- net Net-(C3-Pad2): track 0.00 -> 10.6 mm, vias 0 -> 1
- net Net-(J1-Pad2): track 0.00 -> 9.98 mm, vias 0 -> 1
- net Net-(C2-Pad2): track 0.00 -> 9.24 mm
- net /T_JRST: track 0.00 -> 8.74 mm
- net +5V: track 0.00 -> 7.61 mm, vias 0 -> 1
- net Net-(C10-Pad1): track 0.00 -> 6.57 mm, vias 0 -> 2
- net Net-(Q1-Pad1): track 0.00 -> 6.10 mm
- net Net-(R4-Pad1): track 0.00 -> 5.04 mm
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
Commit message: still gt little bit
Parts:
- moved J3 0.17 mm to (148.3, 99.8)
- moved J4 0.17 mm to (148.3, 99.8)
- moved R14 0.14 mm to (140.7, 109.4)
Routing:
- net /3V3_ST_LINK: track 20.2 -> 89.4 mm, vias 3 -> 12
- net GND: track 47.1 -> 107.0 mm, vias 3 -> 8
- net +5V: track 7.61 -> 15.1 mm, vias 1 -> 2
- net /USB_DM: track 29.8 -> 26.7 mm
- net Net-(D2-Pad1): track 0.00 -> 2.50 mm, vias 0 -> 1
- net Net-(D1-Pad2): track 0.00 -> 2.40 mm, vias 0 -> 1
- net /NRST: track 30.7 -> 32.3 mm
- net /SWIM_RST: track 8.67 -> 7.40 mm
- net /SWIM_IN: track 9.52 -> 10.7 mm
- net /LED_STLINK: track 20.3 -> 19.4 mm
- net /STM_SWDIO_JTMS: track 7.68 -> 8.59 mm
- net /SWIM: track 10.8 -> 11.7 mm
- net /T_SWO: track 14.6 -> 13.9 mm
- net /T_SWDIO_JTMS: track 11.0 -> 10.4 mm
- added copper zone on F.Cu, net /3V3_ST_LINK
- added copper zone on B.Cu, net GND
Other:
- board size 33.6 x 21.2 mm -> 32.1 x 21 mm

Commit message: minor changes
Routing:
- net +5V: track 15.1 -> 16.3 mm
- net Net-(C3-Pad2): track 10.6 -> 9.66 mm
- net /NRST: track 32.3 -> 32.8 mm
Other:
- net class new added: clearance 0.199999, trace_width 0.4, via_dia 0.45, via_drill 0.3

Commit message: done routing
Parts:
- moved D3 0.62 mm to (126.5, 117.1)
- moved C4 0.60 mm to (132.9, 109.5)
- moved R19 0.57 mm to (138.1, 109.4)
- moved R20 0.54 mm to (136.4, 109.4)
- moved R17 0.52 mm to (134.7, 109.4)
- moved R14 0.31 mm to (140.4, 109.4)
- moved C6 0.24 mm to (142.1, 109.5)
- moved J3 0.18 mm to (148.3, 99.6)
- moved J4 0.18 mm to (148.3, 99.6)
- turned R13 to 270 degrees
- turned D2 to 270 degrees
Connections:
- J2 pad 2: /STM_SWCLK_JTCK -> /NRST
- J2 pad 4: /NRST -> /3V3_ST_LINK
- J2 pad 5: /3V3_ST_LINK -> /STM_SWCLK_JTCK
Routing:
- net /3V3_ST_LINK: track 89.0 -> 107.7 mm, vias 12 -> 11
- net /NRST: track 32.8 -> 39.4 mm
- net /LED_STLINK: track 19.4 -> 23.8 mm, vias 5 -> 7
- net /T_RESET: track 16.4 -> 12.4 mm
- net /STM_SWCLK_JTCK: track 6.40 -> 9.78 mm, vias 1 -> 0
- net GND: track 107.0 -> 110.1 mm
- net Net-(C2-Pad2): track 9.19 -> 12.0 mm
- net /T_JTDO: track 11.2 -> 13.5 mm
- net /STM_SWDIO_JTMS: track 8.59 -> 6.80 mm
- net Net-(D3-Pad2): track 2.01 -> 3.59 mm
- net /T_SWIM: track 14.1 -> 14.9 mm
- net +5V: track 16.3 -> 16.9 mm
- net Net-(C3-Pad2): track 9.66 -> 10.3 mm
- net /STLINK_RX: track 12.5 -> 13.1 mm
- net /T_SWDIO_JTMS: track 10.4 -> 10.9 mm
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
Commit message: las version need checking
Parts:
- moved Q1 0.33 mm to (121.2, 100.9)
- moved J3 0.24 mm to (148.4, 99.8)
- moved J4 0.24 mm to (148.4, 99.8)
Routing:
- net /3V3_ST_LINK: track 107.7 -> 117.8 mm
- net /LED_STLINK: track 23.8 -> 24.8 mm
- net /T_RESET: track 12.4 -> 13.5 mm
- net /USB_DP: track 30.6 -> 31.6 mm
- net /T_JTDO: track 13.5 -> 14.3 mm
Other:
- board size 32.1 x 21 mm -> 31.8 x 20.9 mm

Commit message: added label
Parts:
- renumbered J1 to USB
Other:
- board text added: "3V3"
- board text added: "G"
- board text added: "JRST"
- board text added: "JTCK"
- board text added: "JTDI"
- board text added: "JTDO"
- board text added: "JTMS"
- board text added: "PWR"
- board text added: "RST"
- board text added: "RX"
- board text added: "SWM"
- board text added: "SWO"
- board text added: "TX"
- board text added: "nRST"
